Commit message: LiDAR A1M8 support for ROS2 Humble

File: description/lidar.xacro (robot description, xacro)
@@ -6,5 +6,5 @@
         <origin xyz="0.25 0 0.05" rpy="0 0 0"/>
     </joint>
-    <link name="laser_frame">
+    <link name="lidar_link">
         <visual>
             <origin xyz="0 0 0"/>

Commit message: camera support

File: description/lidar.xacro (robot description, xacro)
@@ -3,6 +3,6 @@
     <joint name="laser_joint" type="fixed">
         <parent link="chassis" />
-        <child link="laser_frame" />
-        <origin xyz="0.25 0 0.05" rpy="0 0 0"/>
+        <child link="lidar_link" />
+        <origin xyz="0.25 0 0.175" rpy="0 0 0"/>
     </joint>
     <link name="lidar_link">
@@ -24,9 +24,9 @@
         </xacro:inertial_cylinder>
     </link>
-    <gazebo reference="laser_frame">
+    <gazebo reference="lidar_link">
         <material>Gazebo/Red</material>
         <sensor name="laser" type="ray">
             <pose>0 0 0 0 0 0</pose>
-            <visualize>true</visualize>
+            <visualize>false</visualize>
             <update_rate>10</update_rate>
             <ray>

File: description/robot.urdf.xacro (robot description, xacro)
@@ -4,3 +4,4 @@
     <xacro:include filename="gazebo_control.xacro" />
     <xacro:include filename="lidar.xacro"/>
+    <xacro:include filename="camera.xacro"/>
 </robot>

File: description/robot_core.xacro (robot description, xacro)
@@ -29,17 +29,17 @@
     <link name="chassis">
         <visual>
+            <origin xyz="0.2 0 0.075" />
+            <geometry>
+                <box size="0.4 0.4 0.15" />
+            </geometry>
+            <material name="white" />
+        </visual>
+        <collision>
             <origin xyz="0.2 0 0.015" />
             <geometry>
-                <box size="0.4 0.4 0.03" />
-            </geometry>
-            <material name="white" />
-        </visual>
-        <collision>
-            <origin xyz="0.2 0 0.015" />
-            <geometry>
-                <box size="0.4 0.4 0.03" />
-            </geometry>
-        </collision>
-        <xacro:inertial_box mass="2.0" x="0.4" y="0.4" z="0.03">
+                <box size="0.4 0.4 0.15" />
+            </geometry>
+        </collision>
+        <xacro:inertial_box mass="2.0" x="0.4" y="0.4" z="0.15">
             <origin xyz="0.2 0 0.015" rpy="0 0 0"/>
         </xacro:inertial_box>
