Commit message: support for slam

File: description/robot_core.xacro (robot description, xacro)
@@ -21,5 +21,12 @@
         <!-- You can add visuals and collision properties for the base_link here if needed -->
     </link>
-    <!--CHASSIS LINK-->
+    <joint name="base_footprint_joint" type="fixed">
+        <parent link="base_link"/>
+        <child link="base_footprint"/>
+        <origin xyz="0 0 0" rpy="0 0 0"/>
+    </joint>
+    <link name="base_footprint">
+    </link>
+    <!-- CHASSIS LINK -->
     <joint name="chassis_joint" type="fixed">
         <parent link="base_link"/>
